File: HW/Bettery_Power_Circuit.sch (KiCad schematic (older format))
At the start: 10 parts

Commit message: What did I do?
Parts:
- removed K?: FINDER-40.52, Relays_THT:Relay_DPDT_Finder_40.52, symbol FINDER-40.52
- added K?: FINDER-40.52, Relays_THT:Relay_DPDT_Finder_40.52, symbol FINDER-40.52
Other:
- note added: "CE = HIGH; Battery in parrallel\n"
- note added: "CE = LOW, Battery in series"
- note added: "If SSPNDn = HIGH"
- note added: "If SSPNDn = LOW"
- moved on the sheet: Q?, R?
Changed lines of the file:
@@
 Wire Wire Line
 	5400 2000 5750 2000
-$Comp
-L FINDER-40.52 K?
-U 1 1 5B32EBF2
-P 7000 3050
-F 0 "K?" H 7850 3200 50  0000 L CNN
-F 1 "FINDER-40.52" H 7850 3100 50  0000 L CNN
-F 2 "Relays_THT:Relay_DPDT_Finder_40.52" H 8550 3020 50  0001 C CNN
-F 3 "" H 7000 3050 50  0001 C CNN
-	1    7000 3050
-	-1   0    0    1
-$EndComp
 NoConn ~ 6300 3350
 Wire Wire Line
@@
 L Q_NMOS_DGS Q?
 U 1 1 5B330877
-P 3150 3300
-F 0 "Q?" H 3350 3350 50  0000 L CNN
-F 1 "Q_NMOS_DGS" H 3350 3250 50  0000 L CNN
-F 2 "" H 3350 3400 50  0001 C CNN
-F 3 "" H 3150 3300 50  0001 C CNN
-	1    3150 3300
+P 2900 3400
+F 0 "Q?" H 3100 3450 50  0000 L CNN
+F 1 "Q_NMOS_DGS" H 3100 3350 50  0000 L CNN
+F 2 "" H 3100 3500 50  0001 C CNN
+F 3 "" H 2900 3400 50  0001 C CNN
+	1    2900 3400
 	1    0    0    -1
 $EndComp
@@
 L VBUS #PWR?
 U 1 1 5B330C0A
-P 3250 2900
-F 0 "#PWR?" H 3250 2750 50  0001 C CNN
-F 1 "VBUS" H 3250 3050 50  0000 C CNN
-F 2 "" H 3250 2900 50  0001 C CNN
-F 3 "" H 3250 2900 50  0001 C CNN
-	1    3250 2900
+P 3000 2600
+F 0 "#PWR?" H 3000 2450 50  0001 C CNN
+F 1 "VBUS" H 3000 2750 50  0000 C CNN
+F 2 "" H 3000 2600 50  0001 C CNN
+F 3 "" H 3000 2600 50  0001 C CNN
+	1    3000 2600
 	1    0    0    -1
 $EndComp
@@
 L GND #PWR?
 U 1 1 5B330CC3
-P 3250 4150
-F 0 "#PWR?" H 3250 3900 50  0001 C CNN
-F 1 "GND" H 3250 4000 50  0000 C CNN
-F 2 "" H 3250 4150 50  0001 C CNN
-F 3 "" H 3250 4150 50  0001 C CNN
-	1    3250 4150
-	1    0    0    -1
-$EndComp
-Text HLabel 2750 3300 0    60   Input ~ 0
+P 3000 3750
+F 0 "#PWR?" H 3000 3500 50  0001 C CNN
+F 1 "GND" H 3000 3600 50  0000 C CNN
+F 2 "" H 3000 3750 50  0001 C CNN
+F 3 "" H 3000 3750 50  0001 C CNN
+	1    3000 3750
+	1    0    0    -1
+$EndComp
+Text HLabel 2500 3400 0    60   Input ~ 0
 SSPNDn
 Wire Wire Line
-	2750 3300 2950 3300
+	2500 3400 2700 3400
 $Comp
 L R_Small R?
 U 1 1 5B335E68
-P 3250 3950
-F 0 "R?" H 3280 3970 50  0000 L CNN
-F 1 "10k" H 3280 3910 50  0000 L CNN
-F 2 "" H 3250 3950 50  0001 C CNN
-F 3 "" H 3250 3950 50  0001 C CNN
-	1    3250 3950
-	1    0    0    -1
-$EndComp
-Wire Wire Line
-	3250 2900 3250 3100
-Wire Wire Line
-	3250 3700 3950 3700
-Text Label 3950 3700 2    60   ~ 0
+P 3000 2800
+F 0 "R?" H 3030 2820 50  0000 L CNN
+F 1 "10k" H 3030 2760 50  0000 L CNN
+F 2 "" H 3000 2800 50  0001 C CNN
+F 3 "" H 3000 2800 50  0001 C CNN
+	1    3000 2800
+	1    0    0    -1
+$EndComp
+Wire Wire Line
+	3000 3050 3700 3050
+Text Label 3700 3050 2    60   ~ 0
 CE
 Text Notes 7350 7500 0    60   ~ 0
@@
 Wire Wire Line
 	7750 3700 7500 3700
-Wire Wire Line
-	3250 3500 3250 3850
-Wire Wire Line
-	3250 4150 3250 4050
-Connection ~ 3250 3700
+$Comp
+L FINDER-40.52 K?
+U 1 1 5B342FAB
+P 7000 3050
+F 0 "K?" H 7850 3200 50  0000 L CNN
+F 1 "FINDER-40.52" H 7850 3100 50  0000 L CNN
+F 2 "Relays_THT:Relay_DPDT_Finder_40.52" H 8550 3020 50  0001 C CNN
+F 3 "" H 7000 3050 50  0001 C CNN
+	1    7000 3050
+	-1   0    0    1
+$EndComp
+Wire Wire Line
+	3000 3750 3000 3600
+Wire Wire Line
+	3000 2900 3000 3200
+Connection ~ 3000 3050
+Wire Wire Line
+	3000 2700 3000 2600
+Text Notes 3350 4600 0    60   ~ 0
+If SSPNDn = LOW
+Text Notes 3350 4800 0    60   ~ 0
+If SSPNDn = HIGH
+Text Notes 4450 4600 0    60   ~ 0
+CE = HIGH; Battery in parrallel\n
+Text Notes 4450 4800 0    60   ~ 0
+CE = LOW, Battery in series
+Wire Notes Line
+	3300 4450 3300 4850
+Wire Notes Line
+	3300 4850 5950 4850
+Wire Notes Line
+	5950 4850 5950 4450
+Wire Notes Line
+	5950 4450 3300 4450
+Wire Notes Line
+	4300 4850 4300 4450
+Wire Notes Line
+	3300 4650 5950 4650
 $EndSCHEMATC
