File: HW/USB_DAC.sch (KiCad schematic (older format))
At the start: 43 parts, among them J1 USB_OTG, J2 TP, J3 TP, Q1 Q_NMOS_DGS, U1 PCM2707C, Y1 12 MHz

Commit message: First draft done :100:
Parts:
- removed C1, C2: 100uF, symbol CP1
- removed C10, C5, C6, C8, C9: 1uF, symbol C
- removed C11: 4.7nF, symbol C
- removed C12, C13: 22pF, symbol C
- removed C3, C4: 0.022uF, symbol C
- removed C7: 10uF, symbol CP1
- removed D1: D_TVS, symbol D_TVS
- removed D2: TVS Array, symbol D_TVS_x2_AAC_ALT
- removed D3, D4: LED, symbol LED
- removed J1: USB_OTG, symbol USB_OTG
- removed J2, J3: TP, symbol TEST_1P
- removed L1, L2, L3: 60Ω@100MHz,3A, symbol Ferrite_Bead_Small
- removed Q1: Q_NMOS_DGS, symbol Q_NMOS_DGS
- removed R1, R2: 16, symbol R
- removed R10: NP, symbol R
- removed R11: 1M, symbol R
- removed R12: 0.0, symbol R
- removed R13: 10K, symbol R
- removed R14: 1MΩ, symbol R
- removed R15, R7: 1.5K, symbol R
- removed R16, R17: R, symbol R
- removed R3, R4, R5, R6: 3.3K, symbol R
- removed R8, R9: 22, symbol R
- removed U1: PCM2707C, PCM2707C, symbol PCM2707C
- removed Y1: 12 MHz, symbol Crystal
- added C37, C38: 100uF, symbol CP1
- added C39, C40: 0.022uF, symbol C
- added C41, C42, C44, C45, C46: 1uF, symbol C
- added C43: 10uF, symbol CP1
- added C47: 4.7nF, symbol C
- added C48, C49: 22pF, symbol C
- added D11: LED, 2.1V, 20mA, symbol LED
- added D8: D_TVS, symbol D_TVS
- added D9: TVS Array, symbol D_TVS_x2_AAC_ALT
- added J10, J9: TP, symbol TEST_1P
- added J8: USB_OTG, symbol USB_OTG
- added L10, L8, L9: 60Ω@100MHz,3A, symbol Ferrite_Bead_Small
- added R26, R27: 16, symbol R
- added R28, R29, R30, R31: 3.3K, symbol R
- added R32, R40: 1.5K, symbol R
- added R33, R34: 22, symbol R
- added R35: NP, symbol R
- added R36: 1M, symbol R
- added R37: 0.0, symbol R
- added R38: 10K, symbol R
- added R39: 1MΩ, symbol R
- added R42: 100, symbol R
- added U5: PCM2707C, PCM2707C, symbol PCM2707C
- added Y2: 12 MHz, symbol Crystal
Connections:
- net AGND_DAC: now also C43.2, C44.2, L10.1, U5.1 (PGND)
- net AGND_LR: now also C41.1, C42.1, L8.1, U5.26 (AGNDL), U5.31 (AGNDR)
- net DOUT: now also U5.17 (DOUT)
- net FUNC0: now also U5.5 (FUNC0)
- net FUNC1: now also U5.19 (FUNC1)
- net FUNC2: now also U5.18 (FUNC2)
- net FUNC3: now also U5.4 (FUNC3)
- net GND: now also C45.2, C46.2, C47.2, C48.2, C49.2, D8.1 (A1), D9.3 (common), J8.5 (GND), L10.2, L8.2, R26.2, R27.2, R28.2, R29.2, R30.2, R31.2, R36.2, R37.2, R42.2, U5.20 (DGND), U5.25 (ZGND+)
- net HID0: now also U5.6 (HID0)
- net HID1: now also U5.7 (HID1)
- net HID2: now also U5.8 (HID2)
- net SSPNDn: now also J10.1, R38.2, U5.11 (SSPND)
- net Speaker Op-Amp Circuit/Vin_L: now also C38.2, R31.1
- net Speaker Op-Amp Circuit/Vin_R: now also C37.2, R30.1
- net USB_Dn: now also D9.1 (A1), J8.2 (D-), R34.1
- net USB_Dp: now also D9.2 (A2), J8.3 (D+), R32.2, R33.1
- net VBUS: now also C46.1, D8.2 (A2), L9.1, U5.24 (VBUS)
- net VDD: now also C45.1, D11.2 (A), R32.1, R35.1, R38.1, R40.1, U5.10 (TEST), U5.16 (PSEL), U5.21 (VDD)
- new net: C48.1, R39.2, U5.12 (XTI), Y2.1
- new net: C49.1, R39.1, U5.13 (XTO), Y2.2
- new net: J8.1 (VBUS), L9.2
- new net: C47.1, J8.6 (Shield), R36.1
- new net: C41.2, U5.30 (VCCR)
- new net: C42.2, U5.27 (VCCL)
- new net: R33.2, U5.23 (D+)
- new net: R34.2, U5.22 (D-)
- new net: C37.1, C39.1, R28.1, U5.29 (VOUTR)
- new net: C39.2, R26.1
- new net: C38.1, C40.1, R29.1, U5.28 (VOUTL)
- new net: C40.2, R27.1
- new net: J9.1, R35.2, R37.1, U5.3 (HOST)
- new net: D11.1 (K), R42.1
- new net: R40.2, U5.15 (DT)
- new net: C44.1, U5.2 (VCCP)
- new net: C43.1, U5.32 (VCOM)
Other:
- note removed: "LED Power???\n"
