File: HW/Battery_Power_Circuit.sch (KiCad schematic (older format))
At the start: 22 parts, among them K1 V23105A5001A201, Q2 Q_NMOS_DGS, Q3 Q_NMOS_DGS, Q4 Q_NMOS_DGS, U4 MCP73811, U5 LM2576

Commit message: parts association and some selection
Parts:
- added Q1: Q_NMOS_DGS, TO_SOT_Packages_SMD:SOT-23_Handsoldering, symbol Q_NMOS_DGS
- added R26: 10k, Resistors_SMD:R_0805_HandSoldering, symbol R_Small
- BT1, BT2: footprint (none) -> Connectors_Terminal_Blocks:TerminalBlock_bornier-2_P5.08mm
- C35, C36: footprint (none) -> Capacitors_SMD:C_0805_HandSoldering
- C37, C38: footprint (none) -> Capacitors_SMD:CP_Elec_6.3x5.7
- C39: footprint (none) -> Capacitors_SMD:CP_Elec_6.3x7.7
- D3, D5, D6: footprint (none) -> Diodes_SMD:D_SOD-123
- D7: value LED, 2.1V, 20mA -> LED GREEN; footprint (none) -> Diodes_SMD:D_0805
- L8: footprint (none) -> Inductors_SMD:L_12x12mm_h4.5mm
- L9: value 330uH -> 100uH; footprint (none) -> Inductors_SMD:L_12x12mm_h8mm
- Q2, Q3, Q4: footprint (none) -> TO_SOT_Packages_SMD:SOT-23_Handsoldering
- U4: footprint (none) -> TO_SOT_Packages_SMD:SOT-23-5_HandSoldering
Connections:
- net +5V: now also D7.2 (A), R26.1
- net +BATT: no longer D7.2 (A)
- net GND: now also Q1.3 (S)
- net SSPNDn: now also Q1.2 (G); no longer U5.5 (ENABLEn)
- new net SSPND: Q1.1 (D), R26.2, U5.5 (ENABLEn)
Changed lines of the file:
@@
 EESchema Schematic File Version 2
+LIBS:USB Speaker-rescue
 LIBS:USB-Speaker_Library
 LIBS:power
@@
 F 0 "D5" H 5350 1350 50  0000 C CNN
 F 1 "1N5819" H 5350 1550 50  0000 C CNN
-F 2 "" H 5350 1450 50  0001 C CNN
+F 2 "Diodes_SMD:D_SOD-123" H 5350 1450 50  0001 C CNN
 F 3 "" H 5350 1450 50  0001 C CNN
 	1    5350 1450
@@
 F 0 "U4" H 3950 3200 60  0000 C CNN
 F 1 "MCP73811" H 4150 2300 60  0000 C CNN
-F 2 "" H 3900 2000 60  0001 C CNN
+F 2 "TO_SOT_Packages_SMD:SOT-23-5_HandSoldering" H 3900 2000 60  0001 C CNN
 F 3 "" H 3900 2000 60  0001 C CNN
 	1    3900 2250
@@
 F 0 "C35" H 3110 1720 50  0000 L CNN
 F 1 "1uF" H 3110 1570 50  0000 L CNN
-F 2 "" H 3100 1650 50  0001 C CNN
+F 2 "Capacitors_SMD:C_0805_HandSoldering" H 3100 1650 50  0001 C CNN
 F 3 "" H 3100 1650 50  0001 C CNN
 	1    3100 1650
@@
 F 0 "C36" H 4960 1770 50  0000 L CNN
 F 1 "1uF" H 4960 1620 50  0000 L CNN
-F 2 "" H 4950 1700 50  0001 C CNN
+F 2 "Capacitors_SMD:C_0805_HandSoldering" H 4950 1700 50  0001 C CNN
 F 3 "" H 4950 1700 50  0001 C CNN
 	1    4950 1700
@@
 F 0 "Q2" H 1550 1800 50  0000 L CNN
 F 1 "Q_NMOS_DGS" H 1550 1700 50  0000 L CNN
-F 2 "" H 1550 1850 50  0001 C CNN
+F 2 "TO_SOT_Packages_SMD:SOT-23_Handsoldering" H 1550 1850 50  0001 C CNN
 F 3 "" H 1350 1750 50  0001 C CNN
 	1    1350 1750
@@
 F 0 "Q3" H 6650 3000 50  0000 L CNN
 F 1 "Q_NMOS_DGS" H 6250 3300 50  0000 L CNN
-F 2 "" H 6950 3250 50  0001 C CNN
+F 2 "TO_SOT_Packages_SMD:SOT-23_Handsoldering" H 6950 3250 50  0001 C CNN
 F 3 "" H 6750 3150 50  0001 C CNN
 	1    6750 3150
@@
 F 0 "BT2" H 6050 3400 50  0000 L CNN
 F 1 "18650" H 5950 3200 50  0000 L CNN
-F 2 "" V 5950 3310 50  0001 C CNN
+F 2 "Connectors_Terminal_Blocks:TerminalBlock_bornier-2_P5.08mm" V 5950 3310 50  0001 C CNN
 F 3 "" V 5950 3310 50  0001 C CNN
 	1    5950 3250
@@
 F 0 "BT1" H 6350 2050 50  0000 L CNN
 F 1 "18650" H 6350 1950 50  0000 L CNN
-F 2 "" V 6250 2010 50  0001 C CNN
+F 2 "Connectors_Terminal_Blocks:TerminalBlock_bornier-2_P5.08mm" V 6250 2010 50  0001 C CNN
 F 3 "" V 6250 2010 50  0001 C CNN
 	1    6250 1950
@@
 F 0 "D6" V 7050 2650 50  0000 C CNN
 F 1 "1N4448W" V 7150 2750 50  0000 C CNN
-F 2 "" H 7150 2500 50  0001 C CNN
+F 2 "Diodes_SMD:D_SOD-123" H 7150 2500 50  0001 C CNN
 F 3 "" H 7150 2500 50  0001 C CNN
 	1    7150 2500
@@
 F 0 "Q4" H 2800 3200 50  0000 L CNN
 F 1 "Q_NMOS_DGS" H 2800 3100 50  0000 L CNN
-F 2 "" H 2800 3250 50  0001 C CNN
+F 2 "TO_SOT_Packages_SMD:SOT-23_Handsoldering" H 2800 3250 50  0001 C CNN
 F 3 "" H 2600 3150 50  0001 C CNN
 	1    2600 3150
@@
 AR Path="/5B429541/5B317E48/5B3D11DA" Ref="D14"  Part="1"
 F 0 "D7" V 2750 2500 50  0000 C CNN
-F 1 "LED, 2.1V, 20mA" V 2650 2250 50  0000 C CNN
-F 2 "" H 2700 2700 50  0001 C CNN
+F 1 "LED GREEN" V 2650 2350 50  0000 C CNN
+F 2 "Diodes_SMD:D_0805" H 2700 2700 50  0001 C CNN
 F 3 "" H 2700 2700 50  0001 C CNN
 	1    2700 2700
@@
 	1    0    0    -1
 $EndComp
-$Comp
-L +BATT #PWR115
-U 1 1 5B42F4A3
-P 2700 2450
-AR Path="/5B429541/5B317E48/5B42F4A3" Ref="#PWR115"  Part="1"
-AR Path="/5B42C84F/5B42F4A3" Ref="#PWR053"  Part="1"
-F 0 "#PWR053" H 2700 2300 50  0001 C CNN
-F 1 "+BATT" H 2700 2590 50  0000 C CNN
-F 2 "" H 2700 2450 50  0001 C CNN
-F 3 "" H 2700 2450 50  0001 C CNN
-	1    2700 2450
-	1    0    0    -1
-$EndComp
 Text Notes 3850 1150 0    60   ~ 0
 Battery Charger
 $Comp
-L +BATT #PWR054
+L +BATT #PWR053
 U 1 1 5B442B24
 P 6250 1350
-F 0 "#PWR054" H 6250 1200 50  0001 C CNN
+F 0 "#PWR053" H 6250 1200 50  0001 C CNN
 F 1 "+BATT" H 6250 1490 50  0000 C CNN
 F 2 "" H 6250 1350 50  0001 C CNN
@@
 $EndComp
 $Comp
-L +5V #PWR055
+L +5V #PWR054
 U 1 1 5B4435AD
 P 7100 4500
-F 0 "#PWR055" H 7100 4350 50  0001 C CNN
+F 0 "#PWR054" H 7100 4350 50  0001 C CNN
 F 1 "+5V" H 7100 4640 50  0000 C CNN
 F 2 "" H 7100 4500 50  0001 C CNN
@@
 $EndComp
 $Comp
-L GND #PWR056
+L GND #PWR055
 U 1 1 5B444971
 P 8950 5500
-F 0 "#PWR056" H 8950 5250 50  0001 C CNN
+F 0 "#PWR055" H 8950 5250 50  0001 C CNN
 F 1 "GND" H 8950 5350 50  0000 C CNN
 F 2 "" H 8950 5500 50  0001 C CNN
@@
 $EndComp
 $Comp
-L GND #PWR057
+L GND #PWR056
 U 1 1 5B4449D0
 P 10700 5250
-F 0 "#PWR057" H 10700 5000 50  0001 C CNN
+F 0 "#PWR056" H 10700 5000 50  0001 C CNN
 F 1 "GND" H 10700 5100 50  0000 C CNN
 F 2 "" H 10700 5250 50  0001 C CNN
@@
 	1    0    0    -1
 $EndComp
-Text HLabel 8850 4600 0    60   Input ~ 0
-SSPNDn
 $Comp
 L CP1_Small C37
@@
 F 0 "C37" H 8510 4120 50  0000 L CNN
 F 1 "100uF" H 8510 3970 50  0000 L CNN
-F 2 "" H 8500 4050 50  0001 C CNN
+F 2 "Capacitors_SMD:CP_Elec_6.3x5.7" H 8500 4050 50  0001 C CNN
 F 3 "" H 8500 4050 50  0001 C CNN
 	1    8500 4050
@@
 $EndComp
 $Comp
-L +BATT #PWR058
+L +BATT #PWR057
 U 1 1 5B447866
 P 8500 3750
-F 0 "#PWR058" H 8500 3600 50  0001 C CNN
+F 0 "#PWR057" H 8500 3600 50  0001 C CNN
 F 1 "+BATT" H 8500 3890 50  0000 C CNN
 F 2 "" H 8500 3750 50  0001 C CNN
@@
 $EndComp
 $Comp
-L GND #PWR059
+L GND #PWR058
 U 1 1 5B4478B3
 P 8500 4250
-F 0 "#PWR059" H 8500 4000 50  0001 C CNN
+F 0 "#PWR058" H 8500 4000 50  0001 C CNN
 F 1 "GND" H 8500 4100 50  0000 C CNN
 F 2 "" H 8500 4250 50  0001 C CNN
@@
 F 0 "C39" H 7860 5420 50  0000 L CNN
 F 1 "330uF" H 7860 5270 50  0000 L CNN
-F 2 "" H 7850 5350 50  0001 C CNN
+F 2 "Capacitors_SMD:CP_Elec_6.3x7.7" H 7850 5350 50  0001 C CNN
 F 3 "" H 7850 5350 50  0001 C CNN
 	1    7850 5350
@@
 $EndComp
 $Comp
-L GND #PWR060
+L GND #PWR059
 U 1 1 5B4497AF
 P 7850 5550
-F 0 "#PWR060" H 7850 5300 50  0001 C CNN
+F 0 "#PWR059" H 7850 5300 50  0001 C CNN
 F 1 "GND" H 7850 5400 50  0000 C CNN
 F 2 "" H 7850 5550 50  0001 C CNN
@@
 F 0 "D3" V 8400 5300 50  0000 C CNN
 F 1 "1N5819" V 8500 5400 50  0000 C CNN
-F 2 "" H 8500 5200 50  0001 C CNN
+F 2 "Diodes_SMD:D_SOD-123" H 8500 5200 50  0001 C CNN
 F 3 "" H 8500 5200 50  0001 C CNN
 	1    8500 5200
@@
 	8950 5050 8950 5500
 Wire Wire Line
-	9050 4600 8850 4600
+	8400 4600 9050 4600
 Wire Wire Line
 	8500 4250 8500 4150
@@
 	8500 4750 8500 5050
 $Comp
-L GND #PWR061
+L GND #PWR060
 U 1 1 5B44B4E2
 P 8500 5450
-F 0 "#PWR061" H 8500 5200 50  0001 C CNN
+F 0 "#PWR060" H 8500 5200 50  0001 C CNN
 F 1 "GND" H 8500 5300 50  0000 C CNN
 F 2 "" H 8500 5450 50  0001 C CNN
@@
 P 8150 4750
 F 0 "L9" V 8100 4750 50  0000 C CNN
-F 1 "330uH" V 8225 4750 50  0000 C CNN
-F 2 "" H 8150 4750 50  0001 C CNN
+F 1 "100uH" V 8225 4750 50  0000 C CNN
+F 2 "Inductors_SMD:L_12x12mm_h8mm" H 8150 4750 50  0001 C CNN
 F 3 "" H 8150 4750 50  0001 C CNN
 	1    8150 4750
@@
 F 0 "L8" V 7400 4750 50  0000 C CNN
 F 1 "NP" V 7525 4750 50  0000 C CNN
-F 2 "" H 7450 4750 50  0001 C CNN
+F 2 "Inductors_SMD:L_12x12mm_h4.5mm" H 7450 4750 50  0001 C CNN
 F 3 "" H 7450 4750 50  0001 C CNN
 	1    7450 4750
@@
 F 0 "C38" H 7110 5420 50  0000 L CNN
 F 1 "NP" H 7110 5270 50  0000 L CNN
-F 2 "" H 7100 5350 50  0001 C CNN
+F 2 "Capacitors_SMD:CP_Elec_6.3x5.7" H 7100 5350 50  0001 C CNN
 F 3 "" H 7100 5350 50  0001 C CNN
 	1    7100 5350
@@
 $EndComp
 $Comp
-L GND #PWR062
+L GND #PWR061
 U 1 1 5B451498
 P 7100 5550
-F 0 "#PWR062" H 7100 5300 50  0001 C CNN
+F 0 "#PWR061" H 7100 5300 50  0001 C CNN
 F 1 "GND" H 7100 5400 50  0000 C CNN
 F 2 "" H 7100 5550 50  0001 C CNN
@@
 $Comp
 L LM2576 U5
-U 1 1 5B4544F5
+U 1 1 5B468D35
 P 9250 5350
 F 0 "U5" H 9300 6450 60  0000 C CNN
@@
 	1    0    0    -1
 $EndComp
+$Comp
+L Q_NMOS_DGS Q1
+U 1 1 5B469554
+P 5500 5900
+F 0 "Q1" H 5700 5950 50  0000 L CNN
+F 1 "Q_NMOS_DGS" H 5700 5850 50  0000 L CNN
+F 2 "TO_SOT_Packages_SMD:SOT-23_Handsoldering" H 5700 6000 50  0001 C CNN
+F 3 "" H 5500 5900 50  0001 C CNN
+	1    5500 5900
+	1    0    0    -1
+$EndComp
+$Comp
+L GND #PWR062
+U 1 1 5B469560
+P 5600 6250
+F 0 "#PWR062" H 5600 6000 50  0001 C CNN
+F 1 "GND" H 5600 6100 50  0000 C CNN
+F 2 "" H 5600 6250 50  0001 C CNN
+F 3 "" H 5600 6250 50  0001 C CNN
+	1    5600 6250
+	1    0    0    -1
+$EndComp
+Text HLabel 5100 5900 0    60   Input ~ 0
+SSPNDn
+$Comp
+L R_Small R26
+U 1 1 5B469567
+P 5600 5300
+F 0 "R26" H 5630 5320 50  0000 L CNN
+F 1 "10k" H 5630 5260 50  0000 L CNN
+F 2 "Resistors_SMD:R_0805_HandSoldering" H 5600 5300 50  0001 C CNN
+F 3 "" H 5600 5300 50  0001 C CNN
+	1    5600 5300
+	1    0    0    -1
+$EndComp
+Wire Wire Line
+	5100 5900 5300 5900
+Wire Wire Line
+	5600 5550 6300 5550
+Wire Wire Line
+	5600 6250 5600 6100
+Wire Wire Line
+	5600 5400 5600 5700
+Connection ~ 5600 5550
+Wire Wire Line
+	5600 5200 5600 5100
+Text Label 6300 5550 2    60   ~ 0
+SSPND
+Text Label 8400 4600 0    60   ~ 0
+SSPND
+$Comp
+L +5V #PWR063
+U 1 1 5B47EC4C
+P 5600 5100
+F 0 "#PWR063" H 5600 4950 50  0001 C CNN
+F 1 "+5V" H 5600 5240 50  0000 C CNN
+F 2 "" H 5600 5100 50  0001 C CNN
+F 3 "" H 5600 5100 50  0001 C CNN
+	1    5600 5100
+	1    0    0    -1
+$EndComp
+$Comp
+L +5V #PWR064
+U 1 1 5B47EC9F
+P 2700 2450
+F 0 "#PWR064" H 2700 2300 50  0001 C CNN
+F 1 "+5V" H 2700 2590 50  0000 C CNN
+F 2 "" H 2700 2450 50  0001 C CNN
+F 3 "" H 2700 2450 50  0001 C CNN
+	1    2700 2450
+	1    0    0    -1
+$EndComp
