File: HW/USB Speaker.sch (KiCad schematic (older format))
At the start: 40 parts, among them J1 USB_OTG, J2 TP, J3 TP, U1 PCM2707C, Y1 12 MHz

Commit message: parts association and some selection
Parts:
- C1, C2, C7: footprint (none) -> Capacitors_SMD:CP_Elec_6.3x5.7
- C10, C11, C12, C13, C3, C4, C5, C6, C8, C9: footprint (none) -> Capacitors_SMD:C_0805_HandSoldering
- D1: footprint (none) -> keyboard_parts:D_SC79
- D2: footprint (none) -> TO_SOT_Packages_SMD:SOT-23
- D4: value LED -> LED GREEN; footprint (none) -> Diodes_SMD:D_0805
- J1: footprint (none) -> keyboard_parts:USB_miniB_hirose_5S8
- Y1: footprint (none) -> Crystals:Crystal_HC49-4H_Vertical
Changed lines of the file:
@@
 EESchema Schematic File Version 2
+LIBS:USB Speaker-rescue
 LIBS:USB-Speaker_Library
 LIBS:power
@@
 F 0 "Y1" H 4100 5800 50  0000 C CNN
 F 1 "12 MHz" H 4100 5500 50  0000 C CNN
-F 2 "" H 4100 5650 50  0001 C CNN
+F 2 "Crystals:Crystal_HC49-4H_Vertical" H 4100 5650 50  0001 C CNN
 F 3 "" H 4100 5650 50  0001 C CNN
 	1    4100 5650
@@
 F 0 "C12" H 3875 6150 50  0000 L CNN
 F 1 "22pF" H 3875 5950 50  0000 L CNN
-F 2 "" H 3888 5900 50  0001 C CNN
+F 2 "Capacitors_SMD:C_0805_HandSoldering" H 3888 5900 50  0001 C CNN
 F 3 "" H 3850 6050 50  0001 C CNN
 	1    3850 6050
@@
 F 0 "C13" H 4375 6150 50  0000 L CNN
 F 1 "22pF" H 4375 5950 50  0000 L CNN
-F 2 "" H 4388 5900 50  0001 C CNN
+F 2 "Capacitors_SMD:C_0805_HandSoldering" H 4388 5900 50  0001 C CNN
 F 3 "" H 4350 6050 50  0001 C CNN
 	1    4350 6050
@@
 F 0 "J1" H 8600 3650 50  0000 L CNN
 F 1 "USB_OTG" H 8600 3550 50  0000 L CNN
-F 2 "" H 8950 3150 50  0001 C CNN
+F 2 "keyboard_parts:USB_miniB_hirose_5S8" H 8950 3150 50  0001 C CNN
 F 3 "" H 8950 3150 50  0001 C CNN
 	1    8800 3200
@@
 F 0 "C11" H 9175 3950 50  0000 L CNN
 F 1 "4.7nF" H 9175 3750 50  0000 L CNN
-F 2 "" H 9188 3700 50  0001 C CNN
+F 2 "Capacitors_SMD:C_0805_HandSoldering" H 9188 3700 50  0001 C CNN
 F 3 "" H 9150 3850 50  0001 C CNN
 	1    9150 3850
@@
 F 0 "C10" H 8175 3950 50  0000 L CNN
 F 1 "1uF" H 8175 3750 50  0000 L CNN
-F 2 "" H 8188 3700 50  0001 C CNN
+F 2 "Capacitors_SMD:C_0805_HandSoldering" H 8188 3700 50  0001 C CNN
 F 3 "" H 8150 3850 50  0001 C CNN
 	1    8150 3850
@@
 F 0 "C5" H 3825 2300 50  0000 L CNN
 F 1 "1uF" H 3825 2100 50  0000 L CNN
-F 2 "" H 3838 2050 50  0001 C CNN
+F 2 "Capacitors_SMD:C_0805_HandSoldering" H 3838 2050 50  0001 C CNN
 F 3 "" H 3800 2200 50  0001 C CNN
 	1    3800 2200
@@
 F 0 "C6" H 4425 2300 50  0000 L CNN
 F 1 "1uF" H 4425 2100 50  0000 L CNN
-F 2 "" H 4438 2050 50  0001 C CNN
+F 2 "Capacitors_SMD:C_0805_HandSoldering" H 4438 2050 50  0001 C CNN
 F 3 "" H 4400 2200 50  0001 C CNN
 	1    4400 2200
@@
 F 0 "C8" V 2000 3000 50  0000 L CNN
 F 1 "1uF" V 2100 3000 50  0000 L CNN
-F 2 "" H 2088 3050 50  0001 C CNN
+F 2 "Capacitors_SMD:C_0805_HandSoldering" H 2088 3050 50  0001 C CNN
 F 3 "" H 2050 3200 50  0001 C CNN
 	1    2050 3200
@@
 F 0 "C7" H 1675 2700 50  0000 L CNN
 F 1 "10uF" H 1675 2500 50  0000 L CNN
-F 2 "" H 1650 2600 50  0001 C CNN
+F 2 "Capacitors_SMD:CP_Elec_6.3x5.7" H 1650 2600 50  0001 C CNN
 F 3 "" H 1650 2600 50  0001 C CNN
 	1    1650 2600
@@
 F 0 "C9" H 6325 3950 50  0000 L CNN
 F 1 "1uF" H 6325 3750 50  0000 L CNN
-F 2 "" H 6338 3700 50  0001 C CNN
+F 2 "Capacitors_SMD:C_0805_HandSoldering" H 6338 3700 50  0001 C CNN
 F 3 "" H 6300 3850 50  0001 C CNN
 	1    6300 3850
@@
 F 0 "C3" H 6225 1450 50  0000 L CNN
 F 1 "0.022uF" H 6225 1250 50  0000 L CNN
-F 2 "" H 6238 1200 50  0001 C CNN
+F 2 "Capacitors_SMD:C_0805_HandSoldering" H 6238 1200 50  0001 C CNN
 F 3 "" H 6200 1350 50  0001 C CNN
 	1    6200 1350
@@
 F 0 "C4" H 6675 1450 50  0000 L CNN
 F 1 "0.022uF" H 6675 1250 50  0000 L CNN
-F 2 "" H 6688 1200 50  0001 C CNN
+F 2 "Capacitors_SMD:C_0805_HandSoldering" H 6688 1200 50  0001 C CNN
 F 3 "" H 6650 1350 50  0001 C CNN
 	1    6650 1350
@@
 F 0 "C1" V 7750 950 50  0000 L CNN
 F 1 "100uF" V 7750 550 50  0000 L CNN
-F 2 "" H 7700 850 50  0001 C CNN
+F 2 "Capacitors_SMD:CP_Elec_6.3x5.7" H 7700 850 50  0001 C CNN
 F 3 "" H 7700 850 50  0001 C CNN
 	1    7700 850
@@
 F 0 "C2" V 7750 1200 50  0000 L CNN
 F 1 "100uF" V 7750 800 50  0000 L CNN
-F 2 "" H 7700 1100 50  0001 C CNN
+F 2 "Capacitors_SMD:CP_Elec_6.3x5.7" H 7700 1100 50  0001 C CNN
 F 3 "" H 7700 1100 50  0001 C CNN
 	1    7700 1100
@@
 P 850 5650
 F 0 "D4" H 850 5750 50  0000 C CNN
-F 1 "LED" H 850 5550 50  0000 C CNN
-F 2 "" H 850 5650 50  0001 C CNN
+F 1 "LED GREEN" H 850 5500 50  0000 C CNN
+F 2 "Diodes_SMD:D_0805" H 850 5650 50  0001 C CNN
 F 3 "" H 850 5650 50  0001 C CNN
 	1    850  5650
@@
 F 0 "D2" H 7150 4050 50  0000 C CNN
 F 1 "TVS Array" H 7150 3750 50  0000 C CNN
-F 2 "" V 6800 3950 50  0001 C CNN
+F 2 "TO_SOT_Packages_SMD:SOT-23" V 6800 3950 50  0001 C CNN
 F 3 "" V 6800 3950 50  0001 C CNN
 	1    6900 3800
@@
 F 0 "D1" V 7500 3500 50  0000 C CNN
 F 1 "D_TVS" V 7200 3450 50  0000 C CNN
-F 2 "" H 7400 3650 50  0001 C CNN
+F 2 "keyboard_parts:D_SC79" H 7400 3650 50  0001 C CNN
 F 3 "" H 7400 3650 50  0001 C CNN
 	1    7400 3650
