File: HW/USB_Speaker_page2.sch (KiCad schematic (older format))
At the start: 38 parts, among them J4 TP, J5 TP, J6 TP, U2 BU4S81G2, U3 TPA3137D2

Commit message: First :b:raft 4realz :100:
Other:
- note removed: "Power consumption limit??\n"
Changed lines of the file:
@@
 Wire Wire Line
 	800  4200 800  4000
-Text Notes 800  5150 0    60   ~ 0
-Power consumption limit??\n
 Text Label 3300 4700 0    60   ~ 0
 GVDD

Commit message: 7V Regulator now a 5V buck converter
Parts:
- LS1, LS2: value 2W Speaker -> 4W Speaker
Connections:
- net +BATT renamed +5V
Other:
- note added: "8 Ohm"
- moved on the sheet: J4
Changed lines of the file:
@@
 $Descr A4 11693 8268
 encoding utf-8
-Sheet 2 6
+Sheet 2 3
 Title ""
 Date ""
@@
 AR Path="/5B429541/5B21AA06/5B21D3D0" Ref="LS3"  Part="1"
 F 0 "LS1" H 6700 3500 50  0000 R CNN
-F 1 "2W Speaker" H 7000 3100 50  0000 R CNN
+F 1 "4W Speaker" H 7000 3100 50  0000 R CNN
 F 2 "" H 6700 3200 50  0001 C CNN
 F 3 "" H 6690 3350 50  0001 C CNN
@@
 AR Path="/5B429541/5B21AA06/5B21D3FD" Ref="LS4"  Part="1"
 F 0 "LS2" H 6700 4300 50  0000 R CNN
-F 1 "2W Speaker" H 7050 4700 50  0000 R CNN
+F 1 "4W Speaker" H 7050 4700 50  0000 R CNN
 F 2 "" H 6700 4300 50  0001 C CNN
 F 3 "" H 6690 4450 50  0001 C CNN
@@
 L GND #PWR42
 U 1 1 5B2A5751
-P 2900 5150
+P 2900 5200
 AR Path="/5B42C84D/5B2A5751" Ref="#PWR42"  Part="1"
 AR Path="/5B429541/5B21AA06/5B2A5751" Ref="#PWR99"  Part="1"
-F 0 "#PWR42" H 2900 4900 50  0001 C CNN
-F 1 "GND" H 2900 5000 50  0000 C CNN
-F 2 "" H 2900 5150 50  0001 C CNN
-F 3 "" H 2900 5150 50  0001 C CNN
-	1    2900 5150
+F 0 "#PWR42" H 2900 4950 50  0001 C CNN
+F 1 "GND" H 2900 5050 50  0000 C CNN
+F 2 "" H 2900 5200 50  0001 C CNN
+F 3 "" H 2900 5200 50  0001 C CNN
+	1    2900 5200
 	1    0    0    -1
 $EndComp
@@
 If SSDPNDn or FAULTn are active (LOW), shutdown ampifier
 $Comp
-L +BATT #PWR37
-U 1 1 5B3484B6
-P 1450 3600
-AR Path="/5B42C84D/5B3484B6" Ref="#PWR37"  Part="1"
-AR Path="/5B429541/5B21AA06/5B3484B6" Ref="#PWR94"  Part="1"
-F 0 "#PWR37" H 1450 3450 50  0001 C CNN
-F 1 "+BATT" H 1450 3740 50  0000 C CNN
-F 2 "" H 1450 3600 50  0001 C CNN
-F 3 "" H 1450 3600 50  0001 C CNN
-	1    1450 3600
-	1    0    0    -1
-$EndComp
-$Comp
-L +BATT #PWR30
-U 1 1 5B348527
-P 3400 1650
-AR Path="/5B42C84D/5B348527" Ref="#PWR30"  Part="1"
-AR Path="/5B429541/5B21AA06/5B348527" Ref="#PWR87"  Part="1"
-F 0 "#PWR30" H 3400 1500 50  0001 C CNN
-F 1 "+BATT" H 3400 1790 50  0000 C CNN
-F 2 "" H 3400 1650 50  0001 C CNN
-F 3 "" H 3400 1650 50  0001 C CNN
-	1    3400 1650
-	1    0    0    -1
-$EndComp
-$Comp
-L +BATT #PWR27
-U 1 1 5B348598
-P 6000 1100
-AR Path="/5B42C84D/5B348598" Ref="#PWR27"  Part="1"
-AR Path="/5B429541/5B21AA06/5B348598" Ref="#PWR84"  Part="1"
-F 0 "#PWR27" H 6000 950 50  0001 C CNN
-F 1 "+BATT" H 6000 1240 50  0000 C CNN
-F 2 "" H 6000 1100 50  0001 C CNN
-F 3 "" H 6000 1100 50  0001 C CNN
-	1    6000 1100
-	1    0    0    -1
-$EndComp
-$Comp
-L +BATT #PWR28
-U 1 1 5B348609
-P 7200 1100
-AR Path="/5B42C84D/5B348609" Ref="#PWR28"  Part="1"
-AR Path="/5B429541/5B21AA06/5B348609" Ref="#PWR85"  Part="1"
-F 0 "#PWR28" H 7200 950 50  0001 C CNN
-F 1 "+BATT" H 7200 1240 50  0000 C CNN
-F 2 "" H 7200 1100 50  0001 C CNN
-F 3 "" H 7200 1100 50  0001 C CNN
-	1    7200 1100
-	1    0    0    -1
-$EndComp
-$Comp
-L +BATT #PWR38
-U 1 1 5B3486E0
-P 2900 3950
-AR Path="/5B42C84D/5B3486E0" Ref="#PWR38"  Part="1"
-AR Path="/5B429541/5B21AA06/5B3486E0" Ref="#PWR95"  Part="1"
-F 0 "#PWR38" H 2900 3800 50  0001 C CNN
-F 1 "+BATT" H 2900 4090 50  0000 C CNN
-F 2 "" H 2900 3950 50  0001 C CNN
-F 3 "" H 2900 3950 50  0001 C CNN
-	1    2900 3950
-	1    0    0    -1
-$EndComp
-$Comp
 L BU4S81G2 U2
 U 1 1 5B34B097
@@
 $EndComp
 $Comp
-L +BATT #PWR26
-U 1 1 5B34B179
-P 1750 1100
-AR Path="/5B42C84D/5B34B179" Ref="#PWR26"  Part="1"
-AR Path="/5B429541/5B21AA06/5B34B179" Ref="#PWR83"  Part="1"
-F 0 "#PWR26" H 1750 950 50  0001 C CNN
-F 1 "+BATT" H 1750 1240 50  0000 C CNN
-F 2 "" H 1750 1100 50  0001 C CNN
-F 3 "" H 1750 1100 50  0001 C CNN
-	1    1750 1100
-	1    0    0    -1
-$EndComp
-$Comp
 L C_Small C14
 U 1 1 5B34BCCE
@@
 L TEST_1P J4
 U 1 1 5B3D594F
-P 2700 2000
+P 2700 1950
 AR Path="/5B42C84D/5B3D594F" Ref="J4"  Part="1"
 AR Path="/5B429541/5B21AA06/5B3D594F" Ref="J11"  Part="1"
-F 0 "J4" H 2700 2270 50  0000 C CNN
-F 1 "TP" H 2700 2200 50  0000 C CNN
-F 2 "" H 2900 2000 50  0001 C CNN
-F 3 "" H 2900 2000 50  0001 C CNN
-	1    2700 2000
+F 0 "J4" H 2700 2220 50  0000 C CNN
+F 1 "TP" H 2700 2150 50  0000 C CNN
+F 2 "" H 2900 1950 50  0001 C CNN
+F 3 "" H 2900 1950 50  0001 C CNN
+	1    2700 1950
 	1    0    0    -1
 $EndComp
@@
 	2900 4350 2900 4850
 Wire Wire Line
-	2900 5050 2900 5150
+	2900 5050 2900 5200
 Wire Wire Line
 	3500 5200 3500 4900
@@
 	1400 1500 1400 1450
 Wire Wire Line
-	2700 2300 2700 2000
-Wire Wire Line
-	2700 2000 2300 2000
+	2700 2300 2700 1950
 Wire Wire Line
 	950  4100 950  4000
@@
 Text Label 950  3500 0    60   ~ 0
 GVDD
+Text Notes 7000 3500 0    60   ~ 0
+8 Ohm
+Text Notes 7000 4500 0    60   ~ 0
+8 Ohm
+$Comp
+L +5V #PWR?
+U 1 1 5B454215
+P 1750 1100
+F 0 "#PWR?" H 1750 950 50  0001 C CNN
+F 1 "+5V" H 1750 1240 50  0000 C CNN
+F 2 "" H 1750 1100 50  0001 C CNN
+F 3 "" H 1750 1100 50  0001 C CNN
+	1    1750 1100
+	1    0    0    -1
+$EndComp
+$Comp
+L +5V #PWR?
+U 1 1 5B4543A9
+P 6000 1100
+F 0 "#PWR?" H 6000 950 50  0001 C CNN
+F 1 "+5V" H 6000 1240 50  0000 C CNN
+F 2 "" H 6000 1100 50  0001 C CNN
+F 3 "" H 6000 1100 50  0001 C CNN
+	1    6000 1100
+	1    0    0    -1
+$EndComp
+$Comp
+L +5V #PWR?
+U 1 1 5B454426
+P 7200 1100
+F 0 "#PWR?" H 7200 950 50  0001 C CNN
+F 1 "+5V" H 7200 1240 50  0000 C CNN
+F 2 "" H 7200 1100 50  0001 C CNN
+F 3 "" H 7200 1100 50  0001 C CNN
+	1    7200 1100
+	1    0    0    -1
+$EndComp
+$Comp
+L +5V #PWR?
+U 1 1 5B4545D4
+P 3400 1650
+F 0 "#PWR?" H 3400 1500 50  0001 C CNN
+F 1 "+5V" H 3400 1790 50  0000 C CNN
+F 2 "" H 3400 1650 50  0001 C CNN
+F 3 "" H 3400 1650 50  0001 C CNN
+	1    3400 1650
+	1    0    0    -1
+$EndComp
+$Comp
+L +5V #PWR?
+U 1 1 5B454924
+P 1450 3600
+F 0 "#PWR?" H 1450 3450 50  0001 C CNN
+F 1 "+5V" H 1450 3740 50  0000 C CNN
+F 2 "" H 1450 3600 50  0001 C CNN
+F 3 "" H 1450 3600 50  0001 C CNN
+	1    1450 3600
+	1    0    0    -1
+$EndComp
+$Comp
+L +5V #PWR?
+U 1 1 5B4549A1
+P 2900 3950
+F 0 "#PWR?" H 2900 3800 50  0001 C CNN
+F 1 "+5V" H 2900 4090 50  0000 C CNN
+F 2 "" H 2900 3950 50  0001 C CNN
+F 3 "" H 2900 3950 50  0001 C CNN
+	1    2900 3950
+	1    0    0    -1
+$EndComp
+Wire Wire Line
+	2300 2000 2700 2000
+Connection ~ 2700 2000
 $EndSCHEMATC

Commit message: Buck and fp
Changed buck to one with 3A output. Started fp association
Parts:
- J4, J5, J6: footprint (none) -> Measurement_Points:Measurement_Point_Round-TH_Big
- L4, L5, L6, L7: footprint (none) -> Inductors_SMD:L_0805_HandSoldering
- R18, R19, R20, R21, R22, R23: footprint (none) -> Resistors_SMD:R_0805_HandSoldering
- U3: footprint (none) -> Housings_SSOP:TSSOP-28_4.4x9.7mm_Pitch0.65mm

Commit message: parts association and some selection
Parts:
- removed U2: BU4S81G2, symbol BU4S81G2
- added U2: NC7SZ08, TO_SOT_Packages_SMD:SOT-23-5_HandSoldering, symbol NC7SZ08
- C14, C15, C16, C18, C19, C21, C22, C23, C24, C25, C26, C27, C28, C29, C30, C31, C32, C33, C34: footprint (none) -> Capacitors_SMD:C_0805_HandSoldering
- C17, C20: footprint (none) -> Capacitors_SMD:CP_Elec_6.3x5.7
- LS1, LS2: footprint (none) -> Connectors_Terminal_Blocks:TerminalBlock_bornier-2_P5.08mm
Connections:
- net +5V: now also U2.5 (VCC)
- net FAULTn: now also U2.2 (B)
- net GND: now also U2.3 (GND)
- net SSPNDn: now also U2.1 (A)
- net at J4.1, R18.2, U3.1 (SDn): now also U2.4 (Y)
Changed lines of the file:
@@
 EESchema Schematic File Version 2
+LIBS:USB Speaker-rescue
 LIBS:USB-Speaker_Library
 LIBS:power
@@
 F 0 "LS1" H 6700 3500 50  0000 R CNN
 F 1 "4W Speaker" H 7000 3100 50  0000 R CNN
-F 2 "" H 6700 3200 50  0001 C CNN
+F 2 "Connectors_Terminal_Blocks:TerminalBlock_bornier-2_P5.08mm" H 6700 3200 50  0001 C CNN
 F 3 "" H 6690 3350 50  0001 C CNN
 	1    6700 3400
@@
 F 0 "LS2" H 6700 4300 50  0000 R CNN
 F 1 "4W Speaker" H 7050 4700 50  0000 R CNN
-F 2 "" H 6700 4300 50  0001 C CNN
+F 2 "Connectors_Terminal_Blocks:TerminalBlock_bornier-2_P5.08mm" H 6700 4300 50  0001 C CNN
 F 3 "" H 6690 4450 50  0001 C CNN
 	1    6700 4500
@@
 F 0 "C15" H 5410 1470 50  0000 L CNN
 F 1 "1nF" H 5410 1320 50  0000 L CNN
-F 2 "" H 5400 1400 50  0001 C CNN
+F 2 "Capacitors_SMD:C_0805_HandSoldering" H 5400 1400 50  0001 C CNN
 F 3 "" H 5400 1400 50  0001 C CNN
 	1    5400 1400
@@
 F 0 "C16" H 5710 1470 50  0000 L CNN
 F 1 "100nF" H 5710 1320 50  0000 L CNN
-F 2 "" H 5700 1400 50  0001 C CNN
+F 2 "Capacitors_SMD:C_0805_HandSoldering" H 5700 1400 50  0001 C CNN
 F 3 "" H 5700 1400 50  0001 C CNN
 	1    5700 1400
@@
 F 0 "C17" H 6010 1470 50  0000 L CNN
 F 1 "10uF" H 6010 1320 50  0000 L CNN
-F 2 "" H 6000 1400 50  0001 C CNN
+F 2 "Capacitors_SMD:CP_Elec_6.3x5.7" H 6000 1400 50  0001 C CNN
 F 3 "" H 6000 1400 50  0001 C CNN
 	1    6000 1400
@@
 F 0 "C18" H 6610 1470 50  0000 L CNN
 F 1 "1nF" H 6610 1320 50  0000 L CNN
-F 2 "" H 6600 1400 50  0001 C CNN
+F 2 "Capacitors_SMD:C_0805_HandSoldering" H 6600 1400 50  0001 C CNN
 F 3 "" H 6600 1400 50  0001 C CNN
 	1    6600 1400
@@
 F 0 "C19" H 6910 1470 50  0000 L CNN
 F 1 "100nF" H 6910 1320 50  0000 L CNN
-F 2 "" H 6900 1400 50  0001 C CNN
+F 2 "Capacitors_SMD:C_0805_HandSoldering" H 6900 1400 50  0001 C CNN
 F 3 "" H 6900 1400 50  0001 C CNN
 	1    6900 1400
@@
 F 0 "C20" H 7210 1470 50  0000 L CNN
 F 1 "10uF" H 7210 1320 50  0000 L CNN
-F 2 "" H 7200 1400 50  0001 C CNN
+F 2 "Capacitors_SMD:CP_Elec_6.3x5.7" H 7200 1400 50  0001 C CNN
 F 3 "" H 7200 1400 50  0001 C CNN
 	1    7200 1400
@@
 F 0 "C34" H 3310 5020 50  0000 L CNN
 F 1 "1uF" H 3310 4870 50  0000 L CNN
-F 2 "" H 3300 4950 50  0001 C CNN
+F 2 "Capacitors_SMD:C_0805_HandSoldering" H 3300 4950 50  0001 C CNN
 F 3 "" H 3300 4950 50  0001 C CNN
 	1    3300 4950
@@
 F 0 "C33" H 2910 5020 50  0000 L CNN
 F 1 "1uF" H 2910 4870 50  0000 L CNN
-F 2 "" H 2900 4950 50  0001 C CNN
+F 2 "Capacitors_SMD:C_0805_HandSoldering" H 2900 4950 50  0001 C CNN
 F 3 "" H 2900 4950 50  0001 C CNN
 	1    2900 4950
@@
 F 0 "C21" V 3150 2750 50  0000 L CNN
 F 1 "1uF" V 3150 2500 50  0000 L CNN
-F 2 "" H 3100 2700 50  0001 C CNN
+F 2 "Capacitors_SMD:C_0805_HandSoldering" H 3100 2700 50  0001 C CNN
 F 3 "" H 3100 2700 50  0001 C CNN
 	1    3100 2700
@@
 F 0 "C23" V 3150 3150 50  0000 L CNN
 F 1 "1uF" V 3150 2900 50  0000 L CNN
-F 2 "" H 3100 3100 50  0001 C CNN
+F 2 "Capacitors_SMD:C_0805_HandSoldering" H 3100 3100 50  0001 C CNN
 F 3 "" H 3100 3100 50  0001 C CNN
 	1    3100 3100
@@
 F 0 "C22" V 3150 2950 50  0000 L CNN
 F 1 "1uF" V 3150 2700 50  0000 L CNN
-F 2 "" H 3100 2900 50  0001 C CNN
+F 2 "Capacitors_SMD:C_0805_HandSoldering" H 3100 2900 50  0001 C CNN
 F 3 "" H 3100 2900 50  0001 C CNN
 	1    3100 2900
@@
 F 0 "C25" V 3150 3350 50  0000 L CNN
 F 1 "1uF" V 3150 3100 50  0000 L CNN
-F 2 "" H 3100 3300 50  0001 C CNN
+F 2 "Capacitors_SMD:C_0805_HandSoldering" H 3100 3300 50  0001 C CNN
 F 3 "" H 3100 3300 50  0001 C CNN
 	1    3100 3300
@@
 F 0 "C24" H 5160 3320 50  0000 L CNN
 F 1 "0.22uF" H 5160 3170 50  0000 L CNN
-F 2 "" H 5150 3250 50  0001 C CNN
+F 2 "Capacitors_SMD:C_0805_HandSoldering" H 5150 3250 50  0001 C CNN
 F 3 "" H 5150 3250 50  0001 C CNN
 	1    5150 3250
@@
 F 0 "C32" H 5160 4720 50  0000 L CNN
 F 1 "0.22uF" H 5160 4570 50  0000 L CNN
-F 2 "" H 5150 4650 50  0001 C CNN
+F 2 "Capacitors_SMD:C_0805_HandSoldering" H 5150 4650 50  0001 C CNN
 F 3 "" H 5150 4650 50  0001 C CNN
 	1    5150 4650
@@
 F 0 "C28" H 5160 3720 50  0000 L CNN
 F 1 "0.22uF" H 5160 3570 50  0000 L CNN
-F 2 "" H 5150 3650 50  0001 C CNN
+F 2 "Capacitors_SMD:C_0805_HandSoldering" H 5150 3650 50  0001 C CNN
 F 3 "" H 5150 3650 50  0001 C CNN
 	1    5150 3650
@@
 F 0 "C29" H 5160 4320 50  0000 L CNN
 F 1 "0.22uF" H 5160 4170 50  0000 L CNN
-F 2 "" H 5150 4250 50  0001 C CNN
+F 2 "Capacitors_SMD:C_0805_HandSoldering" H 5150 4250 50  0001 C CNN
 F 3 "" H 5150 4250 50  0001 C CNN
 	1    5150 4250
@@
 F 0 "C26" H 6210 3370 50  0000 L CNN
 F 1 "1uF" H 6210 3220 50  0000 L CNN
-F 2 "" H 6200 3300 50  0001 C CNN
+F 2 "Capacitors_SMD:C_0805_HandSoldering" H 6200 3300 50  0001 C CNN
 F 3 "" H 6200 3300 50  0001 C CNN
 	1    6200 3300
@@
 F 0 "C27" H 6210 3670 50  0000 L CNN
 F 1 "1uF" H 6210 3520 50  0000 L CNN
-F 2 "" H 6200 3600 50  0001 C CNN
+F 2 "Capacitors_SMD:C_0805_HandSoldering" H 6200 3600 50  0001 C CNN
 F 3 "" H 6200 3600 50  0001 C CNN
 	1    6200 3600
@@
 F 0 "C30" H 6210 4370 50  0000 L CNN
 F 1 "1uF" H 6210 4220 50  0000 L CNN
-F 2 "" H 6200 4300 50  0001 C CNN
+F 2 "Capacitors_SMD:C_0805_HandSoldering" H 6200 4300 50  0001 C CNN
 F 3 "" H 6200 4300 50  0001 C CNN
 	1    6200 4300
@@
 F 0 "C31" H 6210 4670 50  0000 L CNN
 F 1 "1uF" H 6210 4520 50  0000 L CNN
-F 2 "" H 6200 4600 50  0001 C CNN
+F 2 "Capacitors_SMD:C_0805_HandSoldering" H 6200 4600 50  0001 C CNN
 F 3 "" H 6200 4600 50  0001 C CNN
 	1    6200 4600
@@
 If SSDPNDn or FAULTn are active (LOW), shutdown ampifier
 $Comp
-L BU4S81G2 U2
-U 1 1 5B34B097
-P 1500 2750
-AR Path="/5B42C84D/5B34B097" Ref="U2"  Part="1"
-AR Path="/5B429541/5B21AA06/5B34B097" Ref="U6"  Part="1"
-F 0 "U2" H 1850 3900 60  0000 C CNN
-F 1 "BU4S81G2" H 2000 3800 60  0000 C CNN
-F 2 "" H 1500 2750 60  0001 C CNN
-F 3 "" H 1500 2750 60  0001 C CNN
-	1    1500 2750
-	1    0    0    -1
-$EndComp
-$Comp
 L C_Small C14
 U 1 1 5B34BCCE
@@
 F 0 "C14" H 1410 1420 50  0000 L CNN
 F 1 "1uF" H 1410 1270 50  0000 L CNN
-F 2 "" H 1400 1350 50  0001 C CNN
+F 2 "Capacitors_SMD:C_0805_HandSoldering" H 1400 1350 50  0001 C CNN
 F 3 "" H 1400 1350 50  0001 C CNN
 	1    1400 1350
@@
 	2300 2000 2700 2000
 Connection ~ 2700 2000
+$Comp
+L NC7SZ08 U2
+U 1 1 5B46B81A
+P 1500 2750
+F 0 "U2" H 1850 3900 60  0000 C CNN
+F 1 "NC7SZ08" H 2000 3800 60  0000 C CNN
+F 2 "TO_SOT_Packages_SMD:SOT-23-5_HandSoldering" H 1500 2750 60  0001 C CNN
+F 3 "" H 1500 2750 60  0001 C CNN
+	1    1500 2750
+	1    0    0    -1
+$EndComp
 $EndSCHEMATC
