File: HW/USB Speaker.kicad_pcb (KiCad board)
At the start: 2 copper layers, 127 x 76.2 mm, 102 parts, among them J1 USB_OTG, J2 TP, J3 TP, J4 TP, J5 TP, J6 TP, K1 V23105A5001A201, Q1 Q_NMOS_DGS, Q2 Q_NMOS_DGS, Q3 Q_NMOS_DGS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

Commit message: initial layout
Parts:
- moved C11 433.7 mm to (193.4, 59.3), turned to 180 degrees
- moved C9 412.9 mm to (179.8, 74.0)
- moved C13 382.2 mm to (195.5, 76.4), turned to 90 degrees
- moved Y1 349.9 mm to (191.8, 82.7), turned to 90 degrees
- moved J1 329.7 mm to (200.5, 60.7), turned to 180 degrees
- moved R11 329.3 mm to (193.3, 57.4), turned to 180 degrees
- moved L2 324.3 mm to (202.9, 64.1), turned to 90 degrees
- moved U1 321.5 mm to (178.3, 80.4), turned to 90 degrees
- moved R14 318.6 mm to (188.0, 80.4), turned to 270 degrees
- moved R15 316.0 mm to (184.7, 76.5), turned to 270 degrees
- moved R9 307.6 mm to (177.6, 70.6), turned to 270 degrees
- moved C37 304.9 mm to (127.7, 153.6)
- moved C12 264.2 mm to (195.5, 84.0), turned to 270 degrees
- moved R8 245.9 mm to (175.8, 70.6), turned to 270 degrees
- moved Q1 229.8 mm to (134.6, 121.9)
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Routing:
- net Net-(D3-Pad1): track 0.00 -> 12.8 mm
- net VBUS: track 0.00 -> 6.83 mm
- net GND: track 0.00 -> 5.39 mm
- net Net-(R9-Pad2): track 0.00 -> 4.62 mm
- net Net-(R8-Pad2): track 0.00 -> 4.60 mm
- net Net-(C13-Pad1): track 0.00 -> 3.18 mm
- net Net-(C12-Pad1): track 0.00 -> 3.18 mm
- added copper zone on F.Cu, net +5V
- added copper zone on F.Cu, net Net-(C39-Pad1)
- added copper zone on F.Cu, net Net-(D3-Pad1)
Other:
- rule trace_min: 0.2 -> 0.127
